File: pcb/_autosave-Macro Pad Pro.kicad_pcb (KiCad board)
At the start: 4 copper layers, 107 x 134 mm, 152 parts, among them J1 USB_C, J2 Conn_02x08_Odd_Even, J3 Conn_02x01, J4 Conn_02x01, SW1 SW_Push_B, SW2 SW_Push_R, U1 RP2040, U3 AP2112K-3.3, U4 USBLC6-2SC6, U6 W25Q128JVS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

Commit message: Changes ready for review
Parts:
- U1: footprint Package_DFN_QFN:QFN-56-1EP_7x7mm_P0.4mm_EP3.2x3.2mm -> Personal:QFN-56-1EP_7x7mm_P0.4mm_EP3.2x3.2mm
- moved C34 0.53 mm to (97.0, 147.1)
- moved C28 0.35 mm to (89.8, 139.4)
Routing:
- net +5V: track 746.9 -> 752.0 mm, vias 35 -> 33
- net +3.3V: track 173.7 -> 176.2 mm, vias 1 -> 0
- net XIN: track 6.59 -> 7.29 mm
- net OLED_CS: track 39.6 -> 39.3 mm, vias 2 -> 1
- net GND: track 24.8 -> 25.0 mm, vias 168 -> 396
- net USB_C_DP: track 6.47 -> 6.40 mm, vias 1 -> 0
