File: pcb/Macro Pad Pro.kicad_pcb (KiCad board)
At the start: 4 copper layers, 107 x 134 mm, 152 parts, among them J1 USB_C, J2 Conn_02x08_Odd_Even, J3 Conn_02x01, J4 Conn_02x01, SW1 SW_Push_B, SW2 SW_Push_R, U1 RP2040, U3 AP2112K-3.3, U4 USBLC6-2SC6, U6 W25Q128JVS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

Commit message: Updated the datalines routing, to be more simple, but longer
Parts:
- removed TP4, TP6: TestPoint, TestPoint:TestPoint_Pad_3.0x3.0mm
- moved R7 4.03 mm to (84.7, 139.9), turned to 180 degrees
- moved C1 3.13 mm to (77.2, 132.8)
- moved U6 2.62 mm to (84.5, 135.6), turned to 180 degrees
- moved R6 1.29 mm to (84.7, 142.0), turned to 180 degrees
Routing:
- net ESD_DM: track 58.6 -> 132.2 mm
- net ESD_DP: track 59.9 -> 131.1 mm
- net +3.3V: track 176.2 -> 150.1 mm, vias 0 -> 1
- net QSPI_SS: track 14.4 -> 9.18 mm
- net QSPI_SCLK: track 11.1 -> 13.9 mm
- net BOOTSEL: track 11.5 -> 13.2 mm
- net QSPI_SD2: track 3.60 -> 4.57 mm
- net GND: vias 396 -> 400
- net Col 4: vias 0 -> 1

Commit message: Changes ready for review
Routing:
- net +3.3V: track 150.1 -> 183.0 mm, vias 1 -> 0
- net GND: vias 400 -> 401
Changed lines of the file:
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@@
 		(tags "Through hole pin header THT 1x02 2.54mm single row")
 		(property "Reference" "J4"
-			(at 0 -2.38 90)
+			(at 0.270573 5.136717 0)
 			(layer "F.SilkS")
 			(effects
@@
 		)
 		(property "Value" "10k"
-			(at 1 -1.3 0)
+			(at -0.05 1.2 0)
 			(layer "F.Fab")
 			(effects
@@
 		)
 		(property "Value" "1k"
-			(at 0 1.399999 90)
+			(at 0.06 -1.29 180)
 			(layer "F.Fab")
 			(effects
@@
 	)
 	(via
+		(at 78.99 136.225)
+		(size 0.5)
+		(drill 0.3)
+		(layers "F.Cu" "B.Cu")
+		(free yes)
+		(net "GND")
+	)
+	(via
 		(at 62.41 126.965)
 		(size 0.5)
@@
 	)
 	(via
-		(at 74.76 143.675)
+		(at 74.63 146.885)
 		(size 0.5)
 		(drill 0.3)
@@
 	)
 	(via
-		(at 73.808868 141.826887)
+		(at 89.49 123.275)
 		(size 0.5)
 		(drill 0.3)
@@
 	)
 	(via
-		(at 74.75 146.405)
+		(at 80.94 131.445)
 		(size 0.5)
 		(drill 0.3)
@@
 	)
 	(via
-		(at 83.65 137.905)
+		(at 84.18 137.675)
 		(size 0.5)
 		(drill 0.3)
@@
 	)
 	(via
-		(at 74.36 145.685)
+		(at 84.32 131.585)
 		(size 0.5)
 		(drill 0.3)
@@
 	)
 	(via
-		(at 78.36 119.365)
+		(at 80.16 119.785)
 		(size 0.5)
 		(drill 0.3)
@@
 	)
 	(segment
+		(start 74.74 113.22)
+		(end 78.12 116.6)
+		(width 0.4)
+		(layer "F.Cu")
+		(net "+3.3V")
+	)
+	(segment
 		(start 112.27 132.335)
 		(end 112.27 133.085)
@@
 	)
 	(segment
+		(start 74.74 113.22)
+		(end 74.975 113.22)
+		(width 0.4)
+		(layer "F.Cu")
+		(net "+3.3V")
+	)
+	(segment
 		(start 95.54 128.975)
 		(end 95.54 130.904811)
@@
 	)
 	(segment
+		(start 78.118 132.845)
+		(end 78.118 136.523)
+		(width 0.4)
+		(layer "F.Cu")
+		(net "+3.3V")
+	)
+	(segment
 		(start 93.221553 141.43953)
 		(end 94.027798 140.633285)
@@
 	)
 	(segment
+		(start 78.12 116.6)
+		(end 78.12 132.843)
+		(width 0.4)
+		(layer "F.Cu")
+		(net "+3.3V")
+	)
+	(segment
 		(start 113.81 122.075)
 		(end 111.65 119.915)
@@
 	)
 	(segment
+		(start 78.12 132.843)
+		(end 78.118 132.845)
+		(width 0.4)
+		(layer "F.Cu")
+		(net "+3.3V")
+	)
+	(segment
 		(start 94.84454 133.4769)
 		(end 94.876326 133.508686)
@@
 	)
 	(segment
+		(start 83.785 138.42)
+		(end 83.785 139.895)
+		(width 0.4)
+		(layer "F.Cu")
+		(net "+3.3V")
+	)
+	(segment
 		(start 112.63 131.975)
 		(end 112.27 132.335)
@@
 	)
 	(segment
+		(start 80.8925 137.4675)
+		(end 82.8325 137.4675)
+		(width 0.4)
+		(layer "F.Cu")
+		(net "+3.3V")
+	)
+	(segment
+		(start 79.0625 137.4675)
+		(end 80.8925 137.4675)
+		(width 0.4)
+		(layer "F.Cu")
+		(net "+3.3V")
+	)
+	(segment
 		(start 94.876326 133.508243)
 		(end 94.498871 133.130788)
@@
 	)
 	(segment
+		(start 78.118 136.523)
+		(end 79.0625 137.4675)
+		(width 0.4)
+		(layer "F.Cu")
+		(net "+3.3V")
+	)
+	(segment
 		(start 118.44 147.915)
 		(end 118.44 135.105)
@@
 	)
 	(segment
+		(start 82.8325 137.4675)
+		(end 83.785 138.42)
+		(width 0.4)
+		(layer "F.Cu")
+		(net "+3.3V")
+	)
+	(segment
 		(start 95.159169 133.225298)
 		(end 95.159169 133.225843)
@@
 		(net "+3.3V")
 	)
-	(via
-		(at 96.17 125.735)
-		(size 0.6)
-		(drill 0.3)
-		(layers "F.Cu" "B.Cu")
-		(net "+3.3V")
-	)
 	(segment
 		(start 59.6 152.25)
@@
 		(width 0.2)
 		(layer "F.Cu")
-		(net "ESD_DM")
-	)
-	(segment
-		(start 45.2 131.765)
-		(end 45.2 131.266471)
-		(width 0.2)
-		(layer "F.Cu")
