File: pcb/Macro Pad Pro.kicad_sch (KiCad schematic)
At the start: 152 parts, among them J1 USB_C, J2 Conn_02x08_Odd_Even, J3 Conn_02x01, J4 Conn_02x01, SW1 SW_Push_B, SW2 SW_Push_R, U1 RP2040, U3 AP2112K-3.3, U4 USBLC6-2SC6, U6 W25Q128JVS, Y1 ABM8-272-T3

Commit message: from work pc
Parts:
- D1, D10, D11, D12, D13, D14, D15, D16, D17, D18, D19, D2, D20, D21, D3, D4, D5, D6, D7, D8, D9, U2, U7: value ~ -> (none)
- LED1, LED10, LED12, LED13, LED14, LED15, LED16, LED17, LED18, LED19, LED2, LED20, LED21, LED3, LED8: footprint PCM_marbastlib-mx:LED_MX_6028R -> Personal:LED_MX_6028R
- LED11, LED4, LED5, LED6, LED7, LED9: footprint PCM_marbastlib-mx:LED_MX_6028R -> Personal:LED_MX_6028R; symbol PCM_marbastlib-mx:MX_SK6812MINI-E -> personal:MX_SK6812MINI-E
- S10, S11, S12, S13, S14, S15, S16, S17, S18, S19, S2, S20, S21, S3, S4, S5, S6, S7, S8, S9: value ~ -> (none); symbol ScottoKeebs:Placeholder_Keyswitch -> personal:Placeholder_Keyswitch
Connections:
- net MCU_DM: no longer R4.2, TP6.1, U4.6
- net MCU_DP: no longer R9.2, TP4.1, U4.4
- new net ESD_DM: R4.2, TP6.1, U4.6
- new net ESD_DP: R9.2, TP4.1, U4.4

Commit message: Changes ready for review
Parts:
- B_LED1, B_LED2, B_LED3, B_LED4, LED1, LED12, LED13, LED14, LED15, LED16, LED17, LED18, LED19, LED2, LED20, LED21, LED3: symbol PCM_marbastlib-mx:MX_SK6812MINI-E -> personal:MX_SK6812MINI-E
- LED10, LED8: footprint Personal:LED_MX_6028R -> PCM_marbastlib-mx:LED_MX_6028R; symbol PCM_marbastlib-mx:MX_SK6812MINI-E -> personal:MX_SK6812MINI-E
Changed lines of the file:
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@@
 	(wire
 		(pts
-			(xy 261.62 232.41) (xy 261.62 233.68)
-		)
-		(stroke
-			(width 0)
-			(type default)
-		)
-	)
-	(wire
-		(pts
 			(xy 88.9 260.35) (xy 87.63 260.35)
 		)
@@
 	)
 	(symbol
-		(lib_id "PCM_marbastlib-mx:MX_SK6812MINI-E")
+		(lib_id "personal:MX_SK6812MINI-E")
 		(at 157.48 172.72 0)
 		(unit 1)
@@
 	)
 	(symbol
-		(lib_id "PCM_marbastlib-mx:MX_SK6812MINI-E")
+		(lib_id "personal:MX_SK6812MINI-E")
 		(at 184.15 31.75 180)
 		(unit 1)
@@
 	)
 	(symbol
-		(lib_id "power:PWR_FLAG")
-		(at 261.62 233.68 180)
-		(unit 1)
-		(body_style 1)
-		(exclude_from_sim no)
-		(in_bom yes)
-		(on_board yes)
-		(in_pos_files yes)
-		(dnp no)
-		(fields_autoplaced yes)
-		(property "Reference" "#FLG04"
-			(at 261.62 235.585 0)
-			(hide yes)
-			(show_name no)
-			(do_not_autoplace no)
-			(effects
-				(font
-					(size 1.27 1.27)
-				)
-			)
-		)
-		(property "Value" "PWR_FLAG"
-			(at 261.62 237.8131 0)
-			(hide yes)
-			(show_name no)
-			(do_not_autoplace no)
-			(effects
-				(font
-					(size 1.27 1.27)
-				)
-			)
-		)
-		(property "Footprint" ""
-			(at 261.62 233.68 0)
-			(hide yes)
-			(show_name no)
-			(do_not_autoplace no)
-			(effects
-				(font
-					(size 1.27 1.27)
-				)
-			)
-		)
-		(property "Datasheet" ""
-			(at 261.62 233.68 0)
-			(hide yes)
-			(show_name no)
-			(do_not_autoplace no)
-			(effects
-				(font
-					(size 1.27 1.27)
-				)
-			)
-		)
-		(property "Description" "Special symbol for telling ERC where power comes from"
-			(at 261.62 233.68 0)
-			(hide yes)
-			(show_name no)
-			(do_not_autoplace no)
-			(effects
-				(font
-					(size 1.27 1.27)
-				)
-			)
-		)
-		(pin "1"
-		)
-		(instances
-			(project "Macro Pad Pro"
-				(path "/92054fa3-5ad0-458e-bd73-acbcf8d11243"
-					(reference "#FLG04")
-					(unit 1)
-				)
-			)
-		)
-	)
-	(symbol
 		(lib_id "Device:D_Small")
 		(at 73.66 110.49 90)
@@
 	)
 	(symbol
-		(lib_id "PCM_marbastlib-mx:MX_SK6812MINI-E")
+		(lib_id "personal:MX_SK6812MINI-E")
 		(at 142.24 106.68 270)
 		(unit 1)
@@
 			)
 		)
-		(property "Footprint" "Personal:LED_MX_6028R"
+		(property "Footprint" "PCM_marbastlib-mx:LED_MX_6028R"
 			(at 142.24 106.68 0)
 			(hide yes)
@@
 	)
 	(symbol
-		(lib_id "PCM_marbastlib-mx:MX_SK6812MINI-E")
+		(lib_id "personal:MX_SK6812MINI-E")
 		(at 157.48 138.43 0)
 		(unit 1)
@@
 	)
 	(symbol
-		(lib_id "PCM_marbastlib-mx:MX_SK6812MINI-E")
+		(lib_id "personal:MX_SK6812MINI-E")
 		(at 302.26 123.19 0)
 		(unit 1)
@@
 	)
 	(symbol
-		(lib_id "PCM_marbastlib-mx:MX_SK6812MINI-E")
+		(lib_id "personal:MX_SK6812MINI-E")
 		(at 142.24 82.55 270)
 		(unit 1)
@@
 			)
 		)
-		(property "Footprint" "Personal:LED_MX_6028R"
+		(property "Footprint" "PCM_marbastlib-mx:LED_MX_6028R"
 			(at 142.24 82.55 0)
 			(hide yes)
@@
 	)
 	(symbol
-		(lib_id "PCM_marbastlib-mx:MX_SK6812MINI-E")
+		(lib_id "personal:MX_SK6812MINI-E")
 		(at 257.81 138.43 0)
 		(mirror y)
@@
 	)
 	(symbol
-		(lib_id "PCM_marbastlib-mx:MX_SK6812MINI-E")
+		(lib_id "personal:MX_SK6812MINI-E")
 		(at 233.68 172.72 0)
 		(unit 1)
@@
 	)
 	(symbol
-		(lib_id "PCM_marbastlib-mx:MX_SK6812MINI-E")
+		(lib_id "personal:MX_SK6812MINI-E")
 		(at 209.55 138.43 0)
 		(mirror y)
@@
 	)
 	(symbol
-		(lib_id "power:+3.3V")
-		(at 261.62 232.41 0)
-		(unit 1)
-		(body_style 1)
-		(exclude_from_sim no)
-		(in_bom yes)
-		(on_board yes)
-		(in_pos_files yes)
-		(dnp no)
-		(fields_autoplaced yes)
-		(property "Reference" "#PWR055"
-			(at 261.62 236.22 0)
-			(hide yes)
-			(show_name no)
-			(do_not_autoplace no)
-			(effects
-				(font
-					(size 1.27 1.27)
-				)
-			)
-		)
-		(property "Value" "+3.3V"
-			(at 261.62 227.33 0)
-			(show_name no)
-			(do_not_autoplace no)
-			(effects
-				(font
-					(size 1.27 1.27)
-				)
-			)
-		)
-		(property "Footprint" ""
-			(at 261.62 232.41 0)
-			(hide yes)
-			(show_name no)
-			(do_not_autoplace no)
-			(effects
-				(font
-					(size 1.27 1.27)
-				)
-			)
-		)
-		(property "Datasheet" ""
-			(at 261.62 232.41 0)
-			(hide yes)
-			(show_name no)
-			(do_not_autoplace no)
-			(effects
-				(font
-					(size 1.27 1.27)
-				)
-			)
-		)
-		(property "Description" "Power symbol creates a global label with name \"+3.3V\""
-			(at 261.62 232.41 0)
-			(hide yes)
-			(show_name no)
-			(do_not_autoplace no)
-			(effects
-				(font
-					(size 1.27 1.27)
-				)
-			)
-		)
-		(pin "1"
-		)
-		(instances
-			(project "Macro Pad Pro"
-				(path "/92054fa3-5ad0-458e-bd73-acbcf8d11243"
-					(reference "#PWR055")
-					(unit 1)
-				)
-			)
-		)
-	)
-	(symbol
 		(lib_id "power:GND")
 		(at 275.59 63.5 0)
@@
 	)
 	(symbol
-		(lib_id "PCM_marbastlib-mx:MX_SK6812MINI-E")
+		(lib_id "personal:MX_SK6812MINI-E")
 		(at 257.81 172.72 0)
 		(unit 1)
@@
 	)
 	(symbol
-		(lib_id "PCM_marbastlib-mx:MX_SK6812MINI-E")
+		(lib_id "personal:MX_SK6812MINI-E")
 		(at 328.93 123.19 0)
 		(unit 1)
@@
 	)
 	(symbol
-		(lib_id "PCM_marbastlib-mx:MX_SK6812MINI-E")
+		(lib_id "personal:MX_SK6812MINI-E")
 		(at 158.75 31.75 180)
 		(unit 1)
@@
 	)
 	(symbol
-		(lib_id "PCM_marbastlib-mx:MX_SK6812MINI-E")
+		(lib_id "personal:MX_SK6812MINI-E")
 		(at 209.55 31.75 180)
 		(unit 1)
@@
 	)
 	(symbol
-		(lib_id "PCM_marbastlib-mx:MX_SK6812MINI-E")
+		(lib_id "personal:MX_SK6812MINI-E")
 		(at 184.15 138.43 0)
 		(mirror y)
@@
 	)
 	(symbol
-		(lib_id "PCM_marbastlib-mx:MX_SK6812MINI-E")
+		(lib_id "personal:MX_SK6812MINI-E")
 		(at 209.55 172.72 0)
 		(unit 1)
@@
 	)
 	(symbol
-		(lib_id "PCM_marbastlib-mx:MX_SK6812MINI-E")
+		(lib_id "personal:MX_SK6812MINI-E")
 		(at 233.68 138.43 0)
 		(mirror y)
@@
 	)
 	(symbol
-		(lib_id "PCM_marbastlib-mx:MX_SK6812MINI-E")
+		(lib_id "personal:MX_SK6812MINI-E")
 		(at 382.27 123.19 0)
 		(unit 1)
@@
 	)
 	(symbol
-		(lib_id "PCM_marbastlib-mx:MX_SK6812MINI-E")
+		(lib_id "personal:MX_SK6812MINI-E")
 		(at 184.15 172.72 0)
 		(unit 1)
@@
 	)
 	(symbol
-		(lib_id "PCM_marbastlib-mx:MX_SK6812MINI-E")
+		(lib_id "personal:MX_SK6812MINI-E")
 		(at 355.6 123.19 0)
 		(unit 1)

Commit message: cleaned up BOM and updated most components with LCSC number and MPN, sent to PCBWay for review
Parts:
- removed J3: Conn_02x01, Connector_PinHeader_2.54mm:PinHeader_1x02_P2.54mm_Vertical, symbol Connector_Generic:Conn_02x01
- removed R16: 10k, Resistor_SMD:R_0805_2012Metric, symbol personal:R_Small
- removed R17: 10k, Resistor_SMD:R_0805_2012Metric, symbol Device:R_Small
- removed R8: 500 ohm, Resistor_SMD:R_0603_1608Metric, symbol Device:R
- removed TP4, TP6: TestPoint, TestPoint:TestPoint_Pad_3.0x3.0mm, symbol Connector:TestPoint
- added R13, R14, R8: 10k, Personal:10k_RESC2012X65N, symbol personal:10k_CRGCQ0805F10K
- B_LED1, B_LED2, B_LED3, B_LED4, J2, LED1, LED11, LED12, LED13, LED14, LED15, LED16, LED17, LED18, LED19, LED2, LED20, LED21, LED3, LED4, LED5, LED6, LED7, LED9, S10, S11, S12, S13, S14, S15, S16, S17, S18, S19, S2, S20, S21, S3, S4, S5, S6, S7, S8, S9, TP10, TP2, TP3, TP8, TP9: now left out of the parts list
- C1, C2, C3, C4, C5, CL1, CL10, CL11, CL12, CL13, CL14, CL15, CL16, CL17, CL18, CL19, CL2, CL20, CL21, CL3, CL4, CL5, CL6, CL7, CL8, CL9: A_max 0.95 -> (none); A_min 0.95 -> (none); A_nom 0.95 -> (none); Check_prices https://www.snapeda.com/parts/CL21B104KBCNNNC/Samsung/view-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 -> (none); D_max 2.1 -> (none); D_min 1.9 -> (none); D_nom 2.0 -> (none); Description_1 0.1 µF ±10% 50V Ceramic Capacitor X7R 0805 (2012 Metric) -> (none); DigiKey_Part_Number 1276-1003-1-ND -> (none); E_max 1.35 -> (none); E_min 1.15 -> (none); E_nom 1.25 -> (none); L1_max 0.7 -> (none); L1_min 0.2 -> (none); L1_nom 0.5 -> (none); LCSC (none) -> C1711; L_max 0.7 -> (none); L_min 0.2 -> (none); L_nom 0.5 -> (none); MANUFACTURER Samsung -> (none); MF Samsung -> (none); MP CL21B104KBCNNNC -> (none); Package SMD-2 Samsung -> (none); STANDARD IPC 7351B -> (none); SnapEDA_Link https://www.snapeda.com/parts/CL21B104KBCNNNC/Samsung/view-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 -> (none)
- C16, C17: A_max 1.8 -> (none); A_min 1.8 -> (none); A_nom 1.8 -> (none); Check_prices https://www.snapeda.com/parts/CL31B106KAHNNNE/Samsung/view-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 -> (none); D_max 3.4 -> (none); D_min 3.0 -> (none); D_nom 3.2 -> (none); Description_1 CL31 Series 10 uF 25 V ±10 % Tolerance X7R SMT Multilayer C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 -> (none); DigiKey_Part_Number 1276-1804-1-ND -> (none); E_max 1.8 -> (none); E_min 1.4 -> (none); E_nom 1.6 -> (none); L1_max 0.8 -> (none); L1_min 0.2 -> (none); L1_nom 0.5 -> (none); LCSC (none) -> C15850; L_max 0.8 -> (none); L_min 0.2 -> (none); L_nom 0.5 -> (none); MANUFACTURER Samsung Electro-Mechanics -> (none); MF Samsung Electro-Mechanics -> (none); MP CL31B106KAHNNNE -> (none); MPN CL31B106KAHNNNE -> CL21A106KAYNNNE; Package SMD-2 Samsung -> (none); STANDARD IPC 7351B -> (none); SnapEDA_Link https://www.snapeda.com/parts/CL31B106KAHNNNE/Samsung/view-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 -> (none)
- C22, C23: A_max 0.65 -> (none); A_min 0.65 -> (none); A_nom 0.65 -> (none); Check_prices https://www.snapeda.com/parts/CL05A105KL5NRNC/Samsung/view-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 -> (none); D_max 1.15 -> (none); D_min 0.85 -> (none); D_nom 1.0 -> (none); Description_1 1 µF ±10% 35V Ceramic Capacitor X5R 0402 (1005 Metric) -> (none); DigiKey_Part_Number 1276-6796-1-ND -> (none); E_max 0.65 -> (none); E_min 0.35 -> (none); E_nom 0.5 -> (none); L1_max 0.35 -> (none); L1_min 0.15 -> (none); L1_nom 0.25 -> (none); LCSC (none) -> C52923; L_max 0.35 -> (none); L_min 0.15 -> (none); L_nom 0.25 -> (none); MANUFACTURER Samsung -> (none); MF Samsung -> (none); MP CL05A105KL5NRNC -> (none); MPN CL21B105KBFNNNE -> CL05A105KA5NQNC; Package SMD-2 Samsung -> (none); STANDARD IPC 7351B -> (none); SnapEDA_Link https://www.snapeda.com/parts/CL05A105KL5NRNC/Samsung/view-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 -> (none)
- C25, C26, C27, C28, C29, C30, C31, C32, C44, C6: A_max 0.55 -> (none); A_min 0.55 -> (none); A_nom 0.55 -> (none); Check_prices https://www.snapeda.com/parts/CL05B104KB5NNNC/Samsung/view-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 -> (none); D_max 1.05 -> (none); D_min 0.95 -> (none); D_nom 1.0 -> (none); Description_1 0.1 µF ±10% 50V Ceramic Capacitor X7R 0402 (1005 Metric) -> (none); DigiKey_Part_Number 1276-CL05B104KB5NNNCCT-ND -> (none); E_max 0.55 -> (none); E_min 0.45 -> (none); E_nom 0.5 -> (none); L1_max 0.35 -> (none); L1_min 0.15 -> (none); L1_nom 0.25 -> (none); LCSC (none) -> C1525; L_max 0.35 -> (none); L_min 0.15 -> (none); L_nom 0.25 -> (none); MANUFACTURER Samsung Electro-Mechanics -> (none); MF Samsung Electro-Mechanics -> (none); MP CL05B104KB5NNNC -> (none); MPN CL21B104KBCNNNC -> CL05B104KO5NNNC; Package SMD-2 Samsung -> (none); Purchase-URL https://www.snapeda.com/api/url_track_click_mouser/?unipart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 -> (none); STANDARD IPC 7351B -> (none); SnapEDA_Link https://www.snapeda.com/parts/CL05B104KB5NNNC/Samsung/view-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 -> (none)
- C33, C34: Availability In Stock -> (none); Check_prices https://www.snapeda.com/parts/885012007052/W%25C3%25BCrth+E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 -> (none); Description_1 WCAP-CSGP General Purpose MLCC; SMT 0805; NP0; 15pF 5%; 50V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 -> (none); LCSC (none) -> C107110; MF Würth Elektronik -> (none); MP 885012007052 -> (none); MPN 885012007052 -> CC0805JRNPO9BN150; Package 0805 Wurth Electronics -> (none); Price None -> (none); Purchase-URL https://www.snapeda.com/api/url_track_click_mouser/?unipart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 -> (none); SnapEDA_Link https://www.snapeda.com/parts/885012007052/W%25C3%25BCrth+E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 -> (none)
- D1, D10, D11, D12, D13, D14, D15, D16, D17, D18, D19, D2, D20, D21, D3, D4, D5, D6, D7, D8, D9: LCSC (none) -> C917030
- F2: MPN (none) -> MF-FSMF050X-2
- J1: Availability In Stock -> (none); Check_prices https://www.snapeda.com/parts/2169900003/Molex/view-part/?r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 -> (none); Description_1 USB-C (USB TYPE-C) USB 2.0 Receptacle Connector 24 (16+8 Du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 -> (none); LCSC (none) -> C3198017; MANUFACTURER Molex -> (none); MAXIMUM_PACKAGE_HEIGHT 2.31 mm -> (none); MF Molex -> (none); MP 2169900003 -> (none); MPN (none) -> 2169900003; PARTREV A1 -> (none); Package None -> (none); Price None -> (none); SNAPEDA_PN 2169900003 -> (none); SnapEDA_Link https://www.snapeda.com/parts/2169900003/Molex/view-part/?r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 -> (none)
- J4: footprint Connector_PinHeader_2.54mm:PinHeader_1x02_P2.54mm_Vertical -> Connector_PinHeader_2.54mm:PinHeader_2x01_P2.54mm_Vertical; now left out of the parts list
- LED10, LED8: footprint PCM_marbastlib-mx:LED_MX_6028R -> Personal:LED_MX_6028R; now left out of the parts list
- R1, R11, R12, R7: Availability In Stock -> (none); Check_prices https://www.snapeda.com/parts/CRGCQ0805F10K/TE+Connectivity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 -> (none); Comment 3-2176341-7 -> (none); Description_1 10 kOhms ±1% 0.125W, 1/8W Chip Resistor 0805 (2012 Metric) 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 -> (none); LCSC (none) -> C17414; MF TE Connectivity -> (none); MP CRGCQ0805F10K -> (none); MPN CRGCQ0805F10K -> 0805W8F1002T5E; Package 2012 TE Connectivity -> (none); Price None -> (none); Purchase-URL https://www.snapeda.com/api/url_track_click_mouser/?unipart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 -> (none); SnapEDA_Link https://www.snapeda.com/parts/CRGCQ0805F10K/TE+Connectivity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 -> (none)
- R10, R6: Availability In Stock -> (none); Check_prices https://www.snapeda.com/parts/CRG0805J1K0/TE+Connectivity+P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 -> (none); Comment 1623327-1 -> (none); Description_1 CRG0805 5% 1K0 -> (none); EU_RoHS_Compliance Compliant with Exemptions -> (none); LCSC (none) -> C95781; MF TE Connectivity -> (none); MP CRG0805J1K0 -> (none); MPN CRG0805J1K0 -> RC0805FR-071KL; Package 0805 -> (none); Power_Rating .125 W -> (none); Price None -> (none); Resistance 1K -> (none); SnapEDA_Link https://www.snapeda.com/parts/CRG0805J1K0/TE+Connectivity+P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 -> (none); Tolerance 5% -> (none); Voltage_Rating 150 V -> (none)
- R15: LCSC C25905 -> C17477; MPN (none) -> 0805W8F0000T5E
- R2, R3: Availability In Stock -> (none); Check_prices https://www.snapeda.com/parts/CRG0805F5K1/TE+Connectivity/v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 -> (none); Comment 1623257-1 -> (none); Description_1 CRG0805 1% 5K1 -> (none); EU_RoHS_Compliance Compliant with Exemptions -> (none); LCSC (none) -> C27834; MF TE Connectivity -> (none); MP CRG0805F5K1 -> (none); MPN CRG0805F5K1 -> 0805W8F5101T5E; Package 0805 -> (none); Power_Rating .125 W -> (none); Price None -> (none); Resistance 5.1K -> (none); SnapEDA_Link https://www.snapeda.com/parts/CRG0805F5K1/TE+Connectivity/v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 -> (none); Tolerance 1% -> (none); Voltage_Rating 150 V -> (none)
- R4, R9: Availability In Stock -> (none); Check_prices https://www.snapeda.com/parts/CRGCQ0805F27R/TE+Connectivity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 -> (none); Comment 2176341-6 -> (none); Description_1 27 Ohms ±1% 0.125W, 1/8W Chip Resistor 0805 (2012 Metric) A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 -> (none); LCSC C25905 -> C17594; MF TE Connectivity -> (none); MP CRGCQ0805F27R -> (none); MPN (none) -> 0805W8F270JT5E; Package 2012 TE Connectivity -> (none); Price None -> (none); Purchase-URL https://www.snapeda.com/api/url_track_click_mouser/?unipart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 -> (none); SnapEDA_Link https://www.snapeda.com/parts/CRGCQ0805F27R/TE+Connectivity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 -> (none)
- R5: value 500 ohm -> 470 ohm; LCSC (none) -> C23179; MPN (none) -> 0603WAF4700T5E
- S1: CREATOR ASHISH -> (none); Check_prices https://www.snapeda.com/parts/PEC11R-4230F-S0024/Bourns/vie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 -> (none); Description_1 Incremental encoder 24 detents 24 pulses | Bourns PEC11R-42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 -> (none); DigiKey_Part_Number PEC11R-4230F-S0024-ND -> (none); MANUFACTURER Bourns -> (none); MF Bourns -> (none); MP PEC11R-4230F-S0024 -> (none); PARTREV 11/23 -> (none); Package None -> (none); SnapEDA_Link https://www.snapeda.com/parts/PEC11R-4230F-S0024/Bourns/vie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 -> (none); now left out of the parts list
- SW1, SW2: footprint Personal:SW_KMR221GLFS -> Button_Switch_SMD:SW_SPST_TL3342; Check_prices https://www.snapeda.com/parts/KMR221G%20LFS/C%2526K/view-pa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 -> (none); Description_1 Switch;Tactile;SPST-NO;OFF-MOM;Top Actuated;1.90mm;2N;0.05A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 -> (none); DigiKey_Part_Number 108-KMR221GLFSCT-ND -> (none); LCSC (none) -> C318884; MANUFACTURER CnK -> (none); MF C&K Components -> (none); MP KMR221G LFS -> (none); MPN (none) -> TS-1187A-B-A-B; Package None -> (none); SnapEDA_Link https://www.snapeda.com/parts/KMR221G%20LFS/C%2526K/view-pa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 -> (none)
- U1: LCSC (none) -> C2040; MPN (none) -> RP2040
- U2: value (none) -> OLED; now left out of the parts list
- U3: LCSC (none) -> C51118
- U4: AVAILABILITY In Stock -> (none); Availability In Stock -> (none); Check_prices https://www.snapeda.com/parts/USBLC6-2SC6/STMicroelectronic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 -> (none); Description_1 17V Clamp 5A (8/20µs) Ipp Tvs Diode Surface Mount SOT-23-6 -> (none); JlcRotOffset -90 -> (none); MF STMicroelectronics -> (none); MP USBLC6-2SC6 -> (none); PACKAGE SOT-23-6 STMicroelectronics -> (none); PRICE None -> (none); PURCHASE-URL https://pricing.snapeda.com/search/part/USBLC6-2SC6/?ref=eda -> (none); Package SOT-23-6 STMicroelectronics -> (none); Price None -> (none); SnapEDA_Link https://www.snapeda.com/parts/USBLC6-2SC6/STMicroelectronic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 -> (none)
- U6: LCSC (none) -> C97521; MPN (none) -> W25Q128JVSIQ
- U7: Check_prices https://www.snapeda.com/parts/SN74AHCT1G125DBVR/Texas+Instr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 -> (none); Description_1 Single 4.5-V to 5.5-V buffer with TTL-compatible CMOS input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 -> (none); DigiKey_Part_Number 296-4708-1-ND -> (none); LCSC (none) -> C7484; MF Texas Instruments -> (none); MP SN74AHCT1G125DBVR -> (none); MPN (none) -> SN74AHCT1G125DBVR; Package SOT-23-5 Texas Instruments -> (none); SnapEDA_Link https://www.snapeda.com/parts/SN74AHCT1G125DBVR/Texas+Instr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 -> (none)
- Y1: Availability In Stock -> (none); CREATOR DIZAR -> (none); Check_prices https://www.snapeda.com/parts/ABM8-272-T3/Abracon/view-part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 -> (none); Description_1 12 MHz ±30ppm Crystal 10pF 50 Ohms 4-SMD, No Lead -> (none); LCSC (none) -> C20625731; MANUFACTURER ABRACON -> (none); MAXIMUM_PACKAGE_HEIGHT 0.8mm -> (none); MF ABRACON -> (none); MP ABM8-272-T3 -> (none); MPN (none) -> ABM8-272-T3; PARTREV 07-29-20 -> (none); Package NON-STANDARD-4 Abracon -> (none); Price None -> (none); Purchase-URL https://www.snapeda.com/api/url_track_click_mouser/?unipart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 -> (none)
Connections:
- net +3.3V: now also R13.2, R14.2
- net GND: now also J2.15 (Pin_15), R8.1
- net LEDS: now also R8.2
- net NRST: now also J2.1 (Pin_1)
- net RCpinA: now also R13.1
- net RCpinB: now also R14.1
- no-connect marks 5 -> 3
Other:
- moved on the sheet: J4, R2
