File: hardware/Macro Pad Pro.kicad_sch (KiCad schematic)
At the start: 149 parts, among them J1 USB_C, J2 Conn_02x08_Odd_Even, J4 Conn_02x01, SW1 SW_Push_B, SW2 SW_Push_R, U1 RP2040, U2 OLED, U3 AP2112K-3.3, U4 USBLC6-2SC6, U6 W25Q128JVS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

Commit message: Fixed ERC component footprint
Parts:
- U4: footprint Personal:SOT95P280X145-6N -> Package_TO_SOT_SMD:SOT-23-6; LCSC (none) -> C7519; MPN (none) -> USBLC6-2SC6
Changed lines of the file:
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@@
 			)
 		)
-		(property "Footprint" "Personal:SOT95P280X145-6N"
+		(property "Footprint" "Package_TO_SOT_SMD:SOT-23-6"
 			(at 323.85 233.68 0)
 			(hide yes)
@@
 			)
 		)
+		(property "MPN" "USBLC6-2SC6"
+			(at 323.85 233.68 0)
+			(hide yes)
+			(show_name no)
+			(do_not_autoplace no)
+			(effects
+				(font
+					(size 1.27 1.27)
+				)
+			)
+		)
+		(property "LCSC" "C7519"
+			(at 323.85 233.68 0)
+			(hide yes)
+			(show_name no)
+			(do_not_autoplace no)
+			(effects
+				(font
+					(size 1.27 1.27)
+				)
+			)
+		)
