File: hardware/Macro Pad Pro.kicad_sch (KiCad schematic)
At the start: 149 parts, among them J1 USB_C, J2 Conn_02x08_Odd_Even, J4 Conn_02x01, SW1 SW_Push_B, SW2 SW_Push_R, U1 RP2040, U2 OLED, U3 AP2112K-3.3, U4 USBLC6-2SC6, U6 W25Q128JVS, Y1 ABM8-272-T3

Commit message: Update PCB design; add production and prototype files
- Update KiCad PCB and schematic (ERC/footprint fixes)
- Regenerate v1.0.0 production package (BOM, positions, designators, netlist)
- Add JLCPCB and new PCBWay production outputs
- Add 10uF 0805 footprint to Personal.pretty and brother.step
- Add prototype design/build photos
- Refresh design backups; remove stale lock files and old PCBWay run

Co-Authored-By: Claude Opus 4.8 <noreply@anthropic.com>
Parts:
- removed F2: 1A, ScottoKeebs_Components:Fuse_0603, symbol Device:Fuse_Small
- C16, C17: footprint Personal:10uF_0805_CAPC3216X180N -> Personal:10uf_0805_CAPC2012X145N
Connections:
- net VBUS: now also R15.1, TP9.1
Changed lines of the file:
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@@
 	)
 	(junction
-		(at 205.74 236.22)
-		(diameter 0)
-		(color 0 0 0 0)
-	)
-	(junction
 		(at 64.77 31.75)
 		(diameter 0)
@@
 		(color 0 0 0 0)
 	)
+	(junction
+		(at 205.74 236.22)
+		(diameter 0)
+		(color 0 0 0 0)
+	)
 	(no_connect
 		(at 134.62 250.19)
@@
 	(wire
 		(pts
-			(xy 191.77 236.22) (xy 195.58 236.22)
+			(xy 191.77 236.22) (xy 205.74 236.22)
 		)
 		(stroke
@@
 	(wire
 		(pts
-			(xy 200.66 236.22) (xy 205.74 236.22)
-		)
-		(stroke
-			(width 0)
-			(type default)
-		)
-	)
-	(wire
-		(pts
 			(xy 149.86 106.68) (xy 161.29 106.68)
 		)
@@
 			)
 		)
-		(property "Footprint" "Personal:10uF_0805_CAPC3216X180N"
+		(property "Footprint" "Personal:10uf_0805_CAPC2012X145N"
 			(at 195.58 267.97 0)
 			(hide yes)
@@
 			)
 		)
-		(property "Footprint" "Personal:10uF_0805_CAPC3216X180N"
+		(property "Footprint" "Personal:10uf_0805_CAPC2012X145N"
 			(at 228.6 267.97 0)
 			(hide yes)
@@
 					(unit 1)
 				)
-			)
-		)
-	)
-	(symbol
-		(lib_id "Device:Fuse_Small")
-		(at 198.12 236.22 0)
-		(unit 1)
-		(body_style 1)
-		(exclude_from_sim no)
-		(in_bom yes)
-		(on_board yes)
-		(in_pos_files yes)
-		(dnp no)
-		(property "Reference" "F2"
-			(at 198.12 231.14 0)
-			(show_name no)
-			(do_not_autoplace no)
-			(effects
-				(font
-					(size 1.27 1.27)
-				)
-			)
-		)
-		(property "Value" "1A"
-			(at 198.12 234.442 0)
-			(show_name no)
-			(do_not_autoplace no)
-			(effects
-				(font
-					(size 1.27 1.27)
-				)
-			)
-		)
-		(property "Footprint" "ScottoKeebs_Components:Fuse_0603"
-			(at 198.12 236.22 0)
-			(hide yes)
-			(show_name no)
-			(do_not_autoplace no)
-			(effects
-				(font
-					(size 1.27 1.27)
-				)
-			)
-		)
-		(property "Datasheet" ""
-			(at 198.12 236.22 0)
-			(hide yes)
-			(show_name no)
-			(do_not_autoplace no)
-			(effects
-				(font
-					(size 1.27 1.27)
-				)
-			)
-		)
-		(property "Description" "Fuse, small symbol"
-			(at 198.12 236.22 0)
-			(hide yes)
-			(show_name no)
-			(do_not_autoplace no)
-			(effects
-				(font
-					(size 1.27 1.27)
-				)
-			)
-		)
-		(property "LCSC" "C210357"
-			(at 198.12 236.22 0)
-			(hide yes)
-			(show_name no)
-			(do_not_autoplace no)
-			(effects
-				(font
-					(size 1.27 1.27)
-				)
-			)
-		)
-		(property "MPN" "MF-FSMF050X-2"
-			(at 198.12 236.22 0)
-			(hide yes)
-			(show_name no)
-			(do_not_autoplace no)
-			(effects
-				(font
-					(size 1.27 1.27)
-				)
-			)
-		)
-		(pin "1"
-		)
-		(pin "2"
-		)
-		(instances
-			(project "Macro Pad Pro"
-				(path "/92054fa3-5ad0-458e-bd73-acbcf8d11243"
-					(reference "F2")
-					(unit 1)
-				)
